Commit message: fix bugs

File: robot_description/urdf/andbot.xacro (robot description, xacro)
@@ -121,5 +121,5 @@
 <!--	<origin xyz="-0.022 0 ${radius_wheel+0.135}" rpy="0 0 0"/>	-->
 <!--	metal model	-->
-<origin xyz="0.07 0 ${radius_wheel+0.135}" rpy="0 0 0"/>
+<origin xyz="0.37 0 ${radius_wheel+0.135}" rpy="0 0 0"/>
   </joint>
 <!--
@@ -878,19 +878,19 @@
       <pose>0 0 0 0 0 0</pose>
       <visualize>true</visualize>
-      <update_rate>5.5</update_rate>
+      <update_rate>10</update_rate>
       <ray>
         <scan>
           <horizontal>
-            <samples>180</samples>
-            <resolution>1</resolution>
-            <min_angle>-1.57</min_angle>
+            <samples>360</samples>
+            <resolution>1</resolution>
+            <min_angle>-3.14</min_angle>
             <!-- -0.0174532925 -->
-            <max_angle>1.57</max_angle>
+            <max_angle>3.14</max_angle>
             <!-- 0.0174532925 -->
           </horizontal>
         </scan>
         <range>
-          <min>0.15</min>
-          <max>6.0</max>
+          <min>0.30</min>
+          <max>12.0</max>
           <resolution>0.01</resolution>
         </range>
